File: led-tube-extensionboard.kicad_sch (KiCad schematic)
At the start: 141 parts, among them Q1 RU20P7C_C605444, Q2 RU20P7C_C605444, Q3 RU20P7C_C605444, SW1 TS-1185EC-C-D-B, SW3 TS-1185EC-C-D-B, U1 QuinLED-ESP32, U10 19-217_R6C-AL1M2VY_3T, U11 SMTSO3015CTJ, U12 SMTSO3015CTJ, U13 SMTSO3015CTJ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

Commit message: regenrate gerber files, add tags
Parts:
- removed BT1, BT2, BT3, BT4: BH-18650-B1BA002, easyeda2kicad:BATTERY-SMD_18650-1S-L77.1-W20.7-1, symbol easyeda2kicad:BH-18650-B1BA002
- removed C14, C41, C51, C52: 10uf, Capacitor_SMD:C_0603_1608Metric_Pad1.08x0.95mm_HandSolder, symbol Device:C
- removed C38, C39, C40, C43, C45, C46, C47, C48: 22uf, Capacitor_SMD:C_0805_2012Metric_Pad1.18x1.45mm_HandSolder, symbol Device:C
- removed C42, C44: 100nf, Capacitor_SMD:C_0603_1608Metric_Pad1.08x0.95mm_HandSolder, symbol Device:C
- removed C49, C50: 2.2uf, Capacitor_SMD:C_0603_1608Metric_Pad1.08x0.95mm_HandSolder, symbol Device:C
- removed C63: CS1E102M-CRI13, easyeda2kicad:CAP-SMD_BD12.5-L13.0-W13.0-FD, symbol easyeda2kicad:CS1E102M-CRI13
- removed F2: BSMD1812-350-16V, easyeda2kicad:F1812, symbol easyeda2kicad:BSMD1812-350-16V
- removed L1: MDA1050-2R2M, easyeda2kicad:IND-SMD_L11.0-W10.0, symbol easyeda2kicad:MDA1050-2R2M
- removed Q1, Q2, Q3: RU20P7C_C605444, easyeda2kicad:SOT-23-3_L2.9-W1.6-P1.90-LS2.8-BR, symbol easyeda2kicad:RU20P7C_C605444
- removed R1: 62, Resistor_SMD:R_0603_1608Metric_Pad0.98x0.95mm_HandSolder, symbol Device:R
- removed R10, R13: 10k, Resistor_SMD:R_0603_1608Metric_Pad0.98x0.95mm_HandSolder, symbol Device:R
- removed R11, R12: 5.1k, Resistor_SMD:R_0603_1608Metric_Pad0.98x0.95mm_HandSolder, symbol Device:R
- removed R2: 113k, Resistor_SMD:R_0603_1608Metric_Pad0.98x0.95mm_HandSolder, symbol Device:R
- removed R3: 0.01, Resistor_SMD:R_0603_1608Metric_Pad0.98x0.95mm_HandSolder, symbol Device:R
- removed R4, R5, R6, R7, R9: 100, Resistor_SMD:R_0603_1608Metric_Pad0.98x0.95mm_HandSolder, symbol Device:R
- removed R8: 82k, Resistor_SMD:R_0603_1608Metric_Pad0.98x0.95mm_HandSolder, symbol Device:R
- removed RT1: TCTR0805F100KF4000T, easyeda2kicad:R0805, symbol easyeda2kicad:TCTR0805F100KF4000T
- removed SW1, SW3: TS-1185EC-C-D-B, footprint:SW-SMD_4P-L3.7-W3.0-P1.50-LS4.7, symbol GLOWINGKITTYPARTS:TS-1185EC-C-D-B
- removed U1: QuinLED-ESP32, quinled:QuinLED-ESP32, symbol quinled:QuinLED-ESP32
- removed U10, U5, U7, U8, U9: 19-217_R6C-AL1M2VY_3T, footprint:LED0603-R-RD, symbol GLOWINGKITTYPARTS:19-217_R6C-AL1M2VY_3T
- removed U12, U13: SMTSO3015CTJ, footprint:SMTSO3030CTJ, symbol GLOWINGKITTYPARTS:SMTSO3015CTJ
- removed U2: U262-161N-4BVC11, footprint:USB-3.1-SMD_U262-161N-4BVC11, symbol GLOWINGKITTYPARTS:U262-161N-4BVC11
- removed U3: IP5328P, easyeda2kicad:QFN-40_L6.0-W6.0-P0.50-BL-EP, symbol easyeda2kicad:IP5328P
- removed U6: SN74AHCT32QPWRQ1, footprint:TSSOP-14_L5.0-W4.4-P0.65-LS6.5-BL, symbol GLOWINGKITTYPARTS:SN74AHCT32QPWRQ1
- removed USB1: MICROXNJ, easyeda2kicad:MICRO-USB-SMD_MICROXNJ, symbol easyeda2kicad:MICROXNJ
- added LED41, LED42, LED43, LED44: XL-5050RGBC-WS2812B, LED_SMD:LED_WS2812B_PLCC4_5.0x5.0mm_P3.2mm, symbol GLOWINGKITTYPARTS:XL-5050RGBC-WS2812B
- C12: value 100nf -> 0.1uF
- C13: value 22uf -> 0.1uF; footprint Capacitor_SMD:C_0805_2012Metric_Pad1.18x1.45mm_HandSolder -> Capacitor_SMD:C_0603_1608Metric_Pad1.08x0.95mm_HandSolder
Connections:
- net +5V: now also C1.2, C12.2, C13.2, LED41.1 (VDD), LED42.1 (VDD), LED43.1 (VDD), LED44.1 (VDD); no longer C1.1
- net GND: now also C1.1, C13.1, LED41.4 (GND), LED42.4 (GND), LED43.4 (GND), LED44.4 (GND); no longer C1.2, C13.2
- net LED DATA NEXT BOARD: no longer names the net of LED40.2 (DO)
- net LED DATA NEXT BOARD: now also LED41.3 (DI); no longer U15.1
- net LED DATA OUT renamed LED DATA IN
- net LED DATA IN: now also U15.1
- removed net VSYS: C12.2, C13.1
- new net: LED42.2 (DO), LED43.3 (DI)
- new net: LED41.2 (DO), LED42.3 (DI)
- new net: LED43.2 (DO), LED44.3 (DI)
Other:
- note removed: "18650 Lithium Battery Cells"
- note removed: "Buttons"
- note removed: "Capacitor behind fuse 1000uF"
- note removed: "ESP32"
- note removed: "Fuse 3.5A 16v"
- note removed: "Level Shifter"
- note removed: "Not entierly sure, if it is needed to pull DMA1 and DPA1 to 5.1k with resistors, or short them, or do nothing to get full 5v 3.1a. Might not place these resistors at first, and test out."
- note removed: "Power"
- note removed: "Power Bank IC"
- note removed: "Power Output from Power Bank IC to Power the 5v rail. This would be a USB-A output port in the reference design."
- note removed: "This is to make sure the datasignal for the LEDs is 5v"
- note removed: "USB-C Port"
- note removed: "mircoUSB Port for Powerbank Input"
- title: led-tube -> led-tube-extensionboard
- moved on the sheet: C10, C11, C17, C18, C19, C20, C21, C22, C23, C24, C25, C26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
